Commit message: Un-normalize line endings in STL files

File: little_red_rover/description/rover/robot.urdf (robot description, URDF)
Before this commit: robot little red rover, 6 links, 5 joints
Links:
- removed link wheel_left
- removed link wheel_right
- added link wheel, mass 0.06046549999362351574; collision mesh filename=package://little_red_rover/description/rover/wheel.stl; visual mesh filename=package://little_red_rover/description/rover/wheel_visual.s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
- added link wheel_2, mass 0.06046549999362351574; collision mesh filename=package://little_red_rover/description/rover/wheel.stl; visual mesh filename=package://little_red_rover/description/rover/wheel_2_visual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
- link robot_body: mass 0.20115864605429473189 -> 0.20097264605429474016
Joints:
- joint base_footprint_frame: origin xyz=0.011199999999999710187 0 -0.043680000000000086813 rpy=-5.9164567891575902922e-31 -6.1629758220391558245e-32 4.8461212225578935465e-32 -> xyz=-0.030479999999999826676 -1.2663481374630691789e-16 -0.036800000000000047951 rpy=-1.570796326794896558 -1.87093529720827402e-49 -1.570796326794896558
- joint base_link_to_base: child robot_body -> wheel
- joint lidar_frame: origin xyz=0.086200000000000123745 -1.3877787807814456755e-17 0.021884999999999994735 rpy=-3.141592653589793116 -3.2417252823925967892e-30 -3.141592653589793116 -> xyz=0.035085000000000268749 -0.075000000000000552336 -0.036800000000000034073 rpy=-1.570796326794896558 -4.8461212225579047131e-31 1.570796326794896558
- joint wheel_left: child wheel_left -> wheel_2; origin xyz=0.011199999999999927028 0.041799999999999955247 -0.013199999999999987785 rpy=-1.5707963267948970021 2.7802557667454690514e-14 -6.5919492087118866803e-16 -> xyz=2.7408630920433552092e-16 -3.5735303605122226145e-16 -0.077600000000000002309 rpy=3.141592653589793116 -8.3992934510864465944e-30 -1.5707963267948976682
- joint wheel_right: child wheel_right -> robot_body; origin xyz=0.01119999999999957141 -0.041800000000000038514 -0.013200000000000263606 rpy=-1.5707963267948961139 6.257321276414477704e-14 3.1415926535897926719 -> xyz=0.011199999999999583553 -0.036800000000000041012 -0.013200000000000263606 rpy=1.570796326794896558 -1.570796326794896558 0; parent robot_body -> wheel

Commit message: Update model with correct child / parent relation

File: little_red_rover/description/rover/robot.urdf (robot description, URDF)
Before this commit: robot little red rover, 6 links, 5 joints
Links:
- link robot_body: mass 0.20097264605429474016 -> 0.2009726460542947124
- link wheel: mass 0.06046549999362351574 -> 0.060465499993623508801
- link wheel_2: mass 0.06046549999362351574 -> 0.060465499993623508801
Joints:
- joint base_footprint_frame: origin xyz=-0.030479999999999826676 -1.2663481374630691789e-16 -0.036800000000000047951 rpy=-1.570796326794896558 -1.87093529720827402e-49 -1.570796326794896558 -> xyz=0.011199999999999710187 0 -0.043680000000000086813 rpy=-5.9164567891575902922e-31 -6.1629758220391558245e-32 4.8461212225578935465e-32
- joint base_link_to_base: child wheel -> robot_body
- joint lidar_frame: origin xyz=0.035085000000000268749 -0.075000000000000552336 -0.036800000000000034073 rpy=-1.570796326794896558 -4.8461212225579047131e-31 1.570796326794896558 -> xyz=0.086200000000000123745 -1.3877787807814456755e-17 0.021884999999999994735 rpy=-3.141592653589793116 -3.2417252823925967892e-30 -3.141592653589793116
- joint wheel_left: child wheel_2 -> wheel; origin xyz=2.7408630920433552092e-16 -3.5735303605122226145e-16 -0.077600000000000002309 rpy=3.141592653589793116 -8.3992934510864465944e-30 -1.5707963267948976682 -> xyz=0.011199999999999940906 0.040799999999999940481 -0.013199999999999989519 rpy=-1.570796326794896558 1.1379786002410102793e-15 -8.3508322388608672319e-30
- joint wheel_right: child robot_body -> wheel_2; origin xyz=0.011199999999999583553 -0.036800000000000041012 -0.013200000000000263606 rpy=1.570796326794896558 -1.570796326794896558 0 -> xyz=0.011199999999999583553 -0.040800000000000023748 -0.013200000000000263606 rpy=-1.570796326794896558 -1.9327092177914794838e-29 4.4289166483876419747e-31; parent wheel -> robot_body

Commit message: Update model for correct wheel orientation

File: little_red_rover/description/rover/robot.urdf (robot description, URDF)
Before this commit: robot little red rover, 6 links, 5 joints
Links:
- link robot_body: mass 0.2009726460542947124 -> 0.20097264605429468465
Joints:
- joint wheel_right: origin xyz=0.011199999999999583553 -0.040800000000000023748 -0.013200000000000263606 rpy=-1.570796326794896558 -1.9327092177914794838e-29 4.4289166483876419747e-31 -> xyz=0.011199999999999583553 -0.040800000000000023748 -0.013200000000000263606 rpy=1.570796326794896558 -1.8488927466117512359e-31 7.0378054251947066516e-30
