Commit message: Lidar driver working, update robot description

File: lrr_description/description/rover/robot.urdf (robot description, URDF)
Before this commit: robot little red rover, 6 links, 5 joints
Links:
- removed link wheel
- removed link wheel_2
- added link wheel_left, mass 0.060465499993623508801; collision mesh filename=package://lrr_description/description/rover/wheel_left.stl; visual mesh filename=package://lrr_description/description/rover/wheel_left_visu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
- added link wheel_right, mass 0.060465499993623932073; collision mesh filename=package://lrr_description/description/rover/wheel_right.stl; visual mesh filename=package://lrr_description/description/rover/wheel_right_vis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
- link robot_body: mass 0.20097264605429468465 -> 0.2009726460542947124
Joints:
- joint wheel_left: child wheel -> wheel_left
- joint wheel_right: child wheel_2 -> wheel_right; origin xyz=0.011199999999999583553 -0.040800000000000023748 -0.013200000000000263606 rpy=1.570796326794896558 -1.8488927466117512359e-31 7.0378054251947066516e-30 -> xyz=0.011200000000000020703 -0.040799999999999912725 -0.013199999999999998193 rpy=-1.570796326794896558 0.57870963485806314885 3.141592653589793116

Commit message: GMapping working

File: lrr_description/description/rover/robot.urdf (robot description, URDF)
Before this commit: robot little red rover, 6 links, 5 joints
Links:
- link wheel_right: mass 0.060465499993623932073 -> 0.060465499993623939012
Joints:
- joint lidar_frame: origin xyz=0.086200000000000123745 -1.3877787807814456755e-17 0.021884999999999994735 rpy=-3.141592653589793116 -3.2417252823925967892e-30 -3.141592653589793116 -> xyz=0.086200000000000123745 0 0.021884999999999994735 rpy=1.4125540584113751048e-29 1.8427297707897078247e-29 -1.0176854567371576776e-30
- joint wheel_right: origin xyz=0.011200000000000020703 -0.040799999999999912725 -0.013199999999999998193 rpy=-1.570796326794896558 0.57870963485806314885 3.141592653589793116 -> xyz=0.011200000000000027642 -0.040799999999999926603 -0.013199999999999998193 rpy=-1.570796326794896558 -0.43939087483637245812 -1.2042149346086100996e-28

Commit message: Fix robot model base_link position, fix bug with concurrent messages

File: lrr_description/description/rover/robot.urdf (robot description, URDF)
Before this commit: robot little_red_rover, 6 links, 5 joints
Links:
- removed link base_footprint
- link wheel_right: mass 0.060465499993623939012 -> 0.060465499993623932073
Joints:
- removed joint base_footprint_frame
- joint lidar_frame: origin xyz=0.086200000000000123745 0 0.021884999999999994735 rpy=1.4125540584113751048e-29 1.8427297707897078247e-29 -1.0176854567371576776e-30 -> xyz=0.074999999999999816813 -3.4694469519534816848e-18 0.065564999999999720726 rpy=3.4502589120532306517e-29 -5.578680289165322067e-30 1.1515748295240288399e-30
- joint wheel_left: origin xyz=0.011199999999999940906 0.040799999999999940481 -0.013199999999999989519 rpy=-1.570796326794896558 1.1379786002410102793e-15 -8.3508322388608672319e-30 -> xyz=3.6203678943636058724e-15 0.040799999999998386169 0.030480000000000645466 rpy=1.570796326794896558 -1.1789999146053913304 3.141592653589793116
- joint wheel_right: origin xyz=0.011200000000000027642 -0.040799999999999926603 -0.013199999999999998193 rpy=-1.570796326794896558 -0.43939087483637245812 -1.2042149346086100996e-28 -> xyz=3.2630148583124013603e-15 -0.040799999999998497191 0.03048000000000037138 rpy=1.570796326794896558 -0.73960903976901759549 -3.141592653589793116

Commit message: Fix robot model base_link position, fix bug with concurrent messages

File: lrr_description/description/rover/robot.urdf (robot description, URDF)
Before this commit: robot little_red_rover, 5 links, 4 joints
Links:
- added link base_footprint, mass 1e-9
- link wheel_right: mass 0.060465499993623932073 -> 0.060465499993623939012
Joints:
- added joint base_footprint_frame: type fixed, parent robot_body, child base_footprint, origin xyz=0.011199999999999710187 0 -0.043680000000000086813 rpy=-5.9164567891575902922e-31 -6.1629758220391558245e-32 4.8461212225578935465e-32, axis 0 0 0
- joint lidar_frame: origin xyz=0.074999999999999816813 -3.4694469519534816848e-18 0.065564999999999720726 rpy=3.4502589120532306517e-29 -5.578680289165322067e-30 1.1515748295240288399e-30 -> xyz=0.086200000000000123745 0 0.021884999999999994735 rpy=1.4125540584113751048e-29 1.8427297707897078247e-29 -1.0176854567371576776e-30
- joint wheel_left: origin xyz=3.6203678943636058724e-15 0.040799999999998386169 0.030480000000000645466 rpy=1.570796326794896558 -1.1789999146053913304 3.141592653589793116 -> xyz=0.011199999999999940906 0.040799999999999940481 -0.013199999999999989519 rpy=-1.570796326794896558 1.1379786002410102793e-15 -8.3508322388608672319e-30
- joint wheel_right: origin xyz=3.2630148583124013603e-15 -0.040799999999998497191 0.03048000000000037138 rpy=1.570796326794896558 -0.73960903976901759549 -3.141592653589793116 -> xyz=0.011200000000000027642 -0.040799999999999926603 -0.013199999999999998193 rpy=-1.570796326794896558 -0.43939087483637245812 -1.2042149346086100996e-28
